File: sensors/ADXL375.kicad_sch (KiCad schematic)
At the start: 5 parts, among them U401 ADXL375

Commit message: Updated references
Parts:
- C401, C405: footprint KwanSystems:SMD_0603 -> Capacitor_SMD:C_0402_1005Metric
- C406: footprint KwanSystems:SMD_0603_pol -> Capacitor_Tantalum_SMD:CP_EIA-3216-18_Kemet-A
- R406: footprint KwanSystems:SMD_0402 -> Resistor_SMD:R_0402_1005Metric
Connections:
- net VCC: now also C401.1
Changed lines of the file:
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@@
   (junction (at 83.82 33.02) (diameter 0) (color 0 0 0 0)
   )
+  (junction (at 101.6 33.02) (diameter 0) (color 0 0 0 0)
+  )
   (junction (at 78.74 55.88) (diameter 0) (color 0 0 0 0)
   )
@@
   (junction (at 101.6 83.82) (diameter 0) (color 0 0 0 0)
   )
-  (junction (at 96.52 38.1) (diameter 0) (color 0 0 0 0)
-  )
   (no_connect (at 93.98 71.12))
-  (wire (pts (xy 93.98 38.1) (xy 96.52 38.1))
-    (stroke (width 0) (type default) (color 0 0 0 0))
-  )
   (wire (pts (xy 74.93 55.88) (xy 78.74 55.88))
     (stroke (width 0) (type default) (color 0 0 0 0))
@@
     (stroke (width 0) (type default) (color 0 0 0 0))
   )
-  (wire (pts (xy 96.52 38.1) (xy 101.6 38.1))
-    (stroke (width 0) (type default) (color 0 0 0 0))
-  )
-  (wire (pts (xy 96.52 43.18) (xy 96.52 38.1))
+  (wire (pts (xy 101.6 33.02) (xy 104.14 33.02))
     (stroke (width 0) (type default) (color 0 0 0 0))
   )
@@
     (stroke (width 0) (type default) (color 0 0 0 0))
   )
-  (wire (pts (xy 83.82 33.02) (xy 104.14 33.02))
+  (wire (pts (xy 83.82 33.02) (xy 101.6 33.02))
     (stroke (width 0) (type default) (color 0 0 0 0))
   )
@@
   )
   (wire (pts (xy 101.6 71.12) (xy 101.6 83.82))
-    (stroke (width 0) (type default) (color 0 0 0 0))
-  )
-  (wire (pts (xy 93.98 38.1) (xy 93.98 43.18))
     (stroke (width 0) (type default) (color 0 0 0 0))
   )
@@
     (effects (font (size 1.524 1.524)) (justify left))
   )
-  (hierarchical_label "SCL" (shape bidirectional) (at 121.92 55.88 0)
+  (hierarchical_label "SCL" (shape input) (at 121.92 55.88 0)
     (effects (font (size 1.524 1.524)) (justify left))
   )
@@
       (effects (font (size 1.143 1.143)) (justify left bottom))
     )
-    (property "Footprint" "KwanSystems:SMD_0402" (id 2) (at 69.977 34.29 0)
+    (property "Footprint" "Resistor_SMD:R_0402_1005Metric" (id 2) (at 69.977 34.29 0)
       (effects (font (size 0.508 0.508)) hide)
     )
@@
     (property "Reference" "C405" (id 0) (at 80.01 41.91 90))
     (property "Value" "100nF" (id 1) (at 77.47 49.53 90))
-    (property "Footprint" "KwanSystems:SMD_0603" (id 2) (at 78.74 45.72 0)
+    (property "Footprint" "Capacitor_SMD:C_0402_1005Metric" (id 2) (at 78.74 45.72 0)
       (effects (font (size 1.27 1.27)) hide)
     )
@@
     (property "Reference" "C401" (id 0) (at 102.87 31.75 90))
     (property "Value" "100nF" (id 1) (at 100.33 39.37 90))
-    (property "Footprint" "KwanSystems:SMD_0603" (id 2) (at 101.6 35.56 0)
+    (property "Footprint" "Capacitor_SMD:C_0402_1005Metric" (id 2) (at 101.6 35.56 0)
       (effects (font (size 1.27 1.27)) hide)
     )
@@
       (effects (font (size 1.27 1.27)) (justify left))
     )
-    (property "Footprint" "KwanSystems:SMD_0603_pol" (id 2) (at 74.93 45.72 0)
-      (effects (font (size 1.27 1.27)) hide)
-    )
+    (property "Footprint" "Capacitor_Tantalum_SMD:CP_EIA-3216-18_Kemet-A" (id 2) (at 74.93 45.72 0)
+      (effects (font (size 1.27 1.27)) hide)
+    )
