File: blocks/Charger.kicad_pcb (KiCad board)
At the start: 2 copper layers, 55.9 x 22.9 mm, 18 parts, among them J801 JST 2mm, U501 MPU9250, U701 3.3V, U801 MCP73831

Commit message: Updated to Kicad 6
Other:
- net class Default removed
