File: blocks/regulator_1v8.kicad_sch (KiCad schematic)
At the start: 3 parts, among them U501 TCR2EF 1.8V

Commit message: Changed to 0603 capacitors
Parts:
- C501, C505: Digikey 399-C0402C105K9PAC7800CT-ND -> 399-C0603C105K4PAC7411CT-ND; Mouser 187-CL05A105KP5NNWC -> 80-C0603C105K4PAC; Number on hand 14+10 -> (none)
- U501: Number on hand 5+3 -> 4
Changed lines of the file:
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@@
       (effects (font (size 1.27 1.27)) hide)
     )
-    (property "Datasheet" "~" (at 114.3 105.41 0)
+    (property "Datasheet" "https://connect.kemet.com:7667/gateway/IntelliData-ComponentDocumentation/1.0/download/datasheet/C0603C105K4PACTU" (at 114.3 105.41 0)
       (effects (font (size 1.27 1.27)) hide)
     )
-    (property "Digikey" "399-C0402C105K9PAC7800CT-ND" (at 114.3 105.41 0)
+    (property "Digikey" "399-C0603C105K4PAC7411CT-ND" (at 114.3 105.41 0)
       (effects (font (size 1.27 1.27)) hide)
     )
@@
       (effects (font (size 1.27 1.27)) hide)
     )
-    (property "Mouser" "187-CL05A105KP5NNWC" (at 114.3 105.41 0)
+    (property "Mouser" "80-C0603C105K4PAC" (at 114.3 105.41 0)
       (effects (font (size 1.27 1.27)) hide)
     )
-    (property "Number on hand" "14+10" (at 114.3 105.41 0)
+    (property "Number on hand" "" (at 114.3 105.41 0)
       (effects (font (size 1.27 1.27)) hide)
     )
@@
         (path "/ba8024d5-8c9d-4001-9766-31acf13004f5/9cdef0f4-d69e-4ec7-af65-50b2b694ea2b"
           (reference "C501") (unit 1)
+        )
+        (path "/ba8024d5-8c9d-4001-9766-31acf13004f5/a0e68691-2daf-412f-ae99-bc89f5381007/f626bd87-a9c2-4f08-af29-d00a1c06cd07"
+          (reference "C801") (unit 1)
         )
       )
@@
       (effects (font (size 1.27 1.27)) hide)
     )
-    (property "Datasheet" "~" (at 144.78 109.22 0)
+    (property "Datasheet" "https://connect.kemet.com:7667/gateway/IntelliData-ComponentDocumentation/1.0/download/datasheet/C0603C105K4PACTU" (at 144.78 109.22 0)
       (effects (font (size 1.27 1.27)) hide)
     )
-    (property "Digikey" "399-C0402C105K9PAC7800CT-ND" (at 144.78 109.22 0)
+    (property "Digikey" "399-C0603C105K4PAC7411CT-ND" (at 144.78 109.22 0)
       (effects (font (size 1.27 1.27)) hide)
     )
@@
       (effects (font (size 1.27 1.27)) hide)
     )
-    (property "Mouser" "187-CL05A105KP5NNWC" (at 144.78 109.22 0)
+    (property "Mouser" "80-C0603C105K4PAC" (at 144.78 109.22 0)
       (effects (font (size 1.27 1.27)) hide)
     )
-    (property "Number on hand" "14+10" (at 144.78 109.22 0)
+    (property "Number on hand" "" (at 144.78 109.22 0)
       (effects (font (size 1.27 1.27)) hide)
     )
@@
         (path "/ba8024d5-8c9d-4001-9766-31acf13004f5/9cdef0f4-d69e-4ec7-af65-50b2b694ea2b"
           (reference "C505") (unit 1)
+        )
+        (path "/ba8024d5-8c9d-4001-9766-31acf13004f5/a0e68691-2daf-412f-ae99-bc89f5381007/f626bd87-a9c2-4f08-af29-d00a1c06cd07"
+          (reference "C805") (unit 1)
         )
       )
@@
       (effects (font (size 1.27 1.27)) hide)
     )
-    (property "Number on hand" "5+3" (at 129.54 96.52 0)
+    (property "Number on hand" "4" (at 129.54 96.52 0)
       (effects (font (size 1.27 1.27)) hide)
     )
@@
           (reference "U501") (unit 1)
         )
+        (path "/ba8024d5-8c9d-4001-9766-31acf13004f5/a0e68691-2daf-412f-ae99-bc89f5381007/f626bd87-a9c2-4f08-af29-d00a1c06cd07"
+          (reference "U801") (unit 1)
+        )
       )

Commit message: Updated number on hand, and added more Digikey/Mouser/Mfg numbers
Parts:
- C501, C505: Number on hand (none) -> 24; Part Number (none) -> C0603C105K4PAC
- U501: Mouser MIC5317-1.8YD5-TR -> 998-MIC5317-1.8YD5TR; Part Number (none) -> MIC5317-1.8YD5-TR
Changed lines of the file:
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@@
       (effects (font (size 1.27 1.27)) hide)
     )
-    (property "Number on hand" "" (at 114.3 105.41 0)
+    (property "Number on hand" "24" (at 114.3 105.41 0)
+      (effects (font (size 1.27 1.27)) hide)
+    )
+    (property "Part Number" "C0603C105K4PAC" (at 114.3 105.41 0)
       (effects (font (size 1.27 1.27)) hide)
     )
@@
       (effects (font (size 1.27 1.27)) hide)
     )
-    (property "Number on hand" "" (at 144.78 109.22 0)
+    (property "Number on hand" "24" (at 144.78 109.22 0)
+      (effects (font (size 1.27 1.27)) hide)
+    )
+    (property "Part Number" "C0603C105K4PAC" (at 144.78 109.22 0)
       (effects (font (size 1.27 1.27)) hide)
     )
@@
       (effects (font (size 1.27 1.27)) hide)
     )
-    (property "Mouser" "MIC5317-1.8YD5-TR" (at 129.54 96.52 0)
+    (property "Mouser" "998-MIC5317-1.8YD5TR" (at 129.54 96.52 0)
       (effects (font (size 1.27 1.27)) hide)
     )
@@
       (effects (font (size 1.27 1.27)) hide)
     )
+    (property "Part Number" "MIC5317-1.8YD5-TR" (at 129.54 96.52 0)
+      (effects (font (size 1.27 1.27)) hide)
+    )
