File: blocks/regulator_1v8.kicad_sch (KiCad schematic)
At the start: 3 parts, among them U501 TCR2EF 1.8V

Commit message: Updated with references to stamp tester
Parts:
- C501, C505: Number on hand 24 -> 12
- U501: Number on hand 4 -> 2
Changed lines of the file:
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@@
       (effects (font (size 1.27 1.27)) hide)
     )
-    (property "Number on hand" "24" (at 114.3 105.41 0)
+    (property "Number on hand" "12" (at 114.3 105.41 0)
       (effects (font (size 1.27 1.27)) hide)
     )
@@
         (path "/ba8024d5-8c9d-4001-9766-31acf13004f5/9cdef0f4-d69e-4ec7-af65-50b2b694ea2b"
           (reference "C501") (unit 1)
-        )
-      )
-      (project "stamp_tester"
-        (path "/bc94e760-f8ab-4abe-bffc-be4558aa8a18/f626bd87-a9c2-4f08-af29-d00a1c06cd07"
-          (reference "C801") (unit 1)
         )
       )
@@
       (effects (font (size 1.27 1.27)) hide)
     )
-    (property "Number on hand" "24" (at 144.78 109.22 0)
+    (property "Number on hand" "12" (at 144.78 109.22 0)
       (effects (font (size 1.27 1.27)) hide)
     )
@@
         (path "/ba8024d5-8c9d-4001-9766-31acf13004f5/9cdef0f4-d69e-4ec7-af65-50b2b694ea2b"
           (reference "C505") (unit 1)
-        )
-      )
-      (project "stamp_tester"
-        (path "/bc94e760-f8ab-4abe-bffc-be4558aa8a18/f626bd87-a9c2-4f08-af29-d00a1c06cd07"
-          (reference "C805") (unit 1)
         )
       )
@@
       (effects (font (size 1.27 1.27)) hide)
     )
-    (property "Number on hand" "4" (at 129.54 96.52 0)
+    (property "Number on hand" "2" (at 129.54 96.52 0)
       (effects (font (size 1.27 1.27)) hide)
     )
@@
         )
       )
-      (project "stamp_tester"
-        (path "/bc94e760-f8ab-4abe-bffc-be4558aa8a18/f626bd87-a9c2-4f08-af29-d00a1c06cd07"
-          (reference "U801") (unit 1)
-        )
-      )
