File: blocks/USB_C_noprot.kicad_sch (KiCad schematic)
At the start: 2 parts, among them J201 USB_C_Receptacle_USB2.0

Commit message: Updated references
Parts:
- J301: renamed from J201; footprint KwanSystems:GCTUSBTypeC_PTH -> KwanSystems:USB_C_Receptacle_GCT_USB4510
- renumbered R2201 to R301
Connections:
- net CC1: now also R301.1 (4); no longer R301.2 (4)
- net CC2: now also R301.2 (4); no longer R301.1 (4)
- net GND: now also R301.4 (3)
Other:
- moved on the sheet: R301A, R301B
Changed lines of the file:
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@@
   (junction (at 111.76 66.04) (diameter 0) (color 0 0 0 0)
+  )
+  (junction (at 119.38 58.42) (diameter 0) (color 0 0 0 0)
   )
   (junction (at 120.65 50.8) (diameter 0) (color 0 0 0 0)
@@
     (stroke (width 0) (type default))
   )
+  (wire (pts (xy 119.38 55.88) (xy 119.38 58.42))
+    (stroke (width 0) (type default))
+  )
   (wire (pts (xy 111.76 68.58) (xy 125.73 68.58))
     (stroke (width 0) (type default))
   )
-  (wire (pts (xy 119.38 55.88) (xy 119.38 88.9))
-    (stroke (width 0) (type default))
-  )
   (wire (pts (xy 111.76 66.04) (xy 125.73 66.04))
+    (stroke (width 0) (type default))
+  )
+  (wire (pts (xy 119.38 58.42) (xy 119.38 88.9))
     (stroke (width 0) (type default))
   )
@@
   (symbol (lib_id "Connector:USB_C_Receptacle_USB2.0") (at 96.52 66.04 0) (unit 1)
     (in_bom yes) (on_board yes) (dnp no)
-    (property "Reference" "J201" (at 99.2378 44.0182 0)
+    (property "Reference" "J301" (at 99.2378 44.0182 0)
       (effects (font (size 1.27 1.27)))
     )
@@
       (effects (font (size 1.27 1.27)))
     )
-    (property "Footprint" "KwanSystems:GCTUSBTypeC_PTH" (at 100.33 66.04 0)
+    (property "Footprint" "KwanSystems:USB_C_Receptacle_GCT_USB4510" (at 100.33 66.04 0)
       (effects (font (size 1.27 1.27)) hide)
     )
@@
     (pin "S1")
     (instances
+      (project "Naninator32u4"
+        (path "/ba1a019e-3acf-4680-bf69-4a14e392b0f8/db3c602a-4181-4312-837d-35d7c3586816"
+          (reference "J301") (unit 1)
+        )
+      )
       (project "Naninator"
         (path "/d855b238-2442-4e65-b657-8cbe334057c3/00000000-0000-0000-0000-00005f5cf167/00000000-0000-0000-0000-00005f690bf7"
@@
     (pin "1")
     (instances
+      (project "Naninator32u4"
+        (path "/ba1a019e-3acf-4680-bf69-4a14e392b0f8/db3c602a-4181-4312-837d-35d7c3586816"
+          (reference "#FLG0102") (unit 1)
+        )
+      )
       (project "Naninator"
         (path "/d855b238-2442-4e65-b657-8cbe334057c3/00000000-0000-0000-0000-00005f5cf167/00000000-0000-0000-0000-00005f690bf7"
@@
     )
   )
-  (symbol (lib_id "KwanSystems:RP2") (at 116.84 58.42 0) (unit 1)
-    (in_bom yes) (on_board yes) (dnp no)
-    (property "Reference" "R2201" (at 123.19 58.42 0)
+  (symbol (lib_id "KwanSystems:RP2") (at 116.84 55.88 0) (unit 1)
+    (in_bom yes) (on_board yes) (dnp no)
+    (property "Reference" "R301" (at 123.19 55.88 0)
       (effects (font (size 1.143 1.143)))
     )
@@
       (effects (font (size 1.143 1.143)))
     )
-    (property "Footprint" "KwanSystems:R_Array_Convex_2x0402" (at 118.237 54.61 0)
+    (property "Footprint" "KwanSystems:R_Array_Convex_2x0402" (at 118.237 52.07 0)
       (effects (font (size 0.508 0.508)) hide)
     )
-    (property "Datasheet" "" (at 127.635 66.04 0)
+    (property "Datasheet" "" (at 127.635 63.5 0)
       (effects (font (size 1.524 1.524)) hide)
     )
@@
     (pin "3")
     (instances
+      (project "Naninator32u4"
+        (path "/ba1a019e-3acf-4680-bf69-4a14e392b0f8/db3c602a-4181-4312-837d-35d7c3586816"
+          (reference "R301") (unit 1)
+        )
+      )
       (project "Naninator"
         (path "/d855b238-2442-4e65-b657-8cbe334057c3/00000000-0000-0000-0000-00005f5cf167/00000000-0000-0000-0000-00005f690bf7"
@@
     )
   )
-  (symbol (lib_id "KwanSystems:RP2") (at 116.84 55.88 0) (unit 2)
-    (in_bom yes) (on_board yes) (dnp no)
-    (property "Reference" "R2201" (at 123.19 55.88 0)
+  (symbol (lib_id "KwanSystems:RP2") (at 116.84 58.42 0) (unit 2)
+    (in_bom yes) (on_board yes) (dnp no)
+    (property "Reference" "R301" (at 123.19 58.42 0)
       (effects (font (size 1.143 1.143)))
     )
@@
       (effects (font (size 1.143 1.143)))
     )
-    (property "Footprint" "KwanSystems:R_Array_Convex_2x0402" (at 118.237 52.07 0)
+    (property "Footprint" "KwanSystems:R_Array_Convex_2x0402" (at 118.237 54.61 0)
       (effects (font (size 0.508 0.508)) hide)
     )
-    (property "Datasheet" "" (at 127.635 63.5 0)
+    (property "Datasheet" "" (at 127.635 66.04 0)
       (effects (font (size 1.524 1.524)) hide)
     )
@@
     (pin "3")
     (instances
-      (project "Naninator"
-        (path "/d855b238-2442-4e65-b657-8cbe334057c3/00000000-0000-0000-0000-00005f5cf167/00000000-0000-0000-0000-00005f690bf7"
+      (project "Naninator32u4"
+        (path "/ba1a019e-3acf-4680-bf69-4a14e392b0f8/db3c602a-4181-4312-837d-35d7c3586816"
+          (reference "R301") (unit 2)
+        )
+      )
+      (project "Naninator"
+        (path "/d855b238-2442-4e65-b657-8cbe334057c3/00000000-0000-0000-0000-00005f5cf167/00000000-0000-0000-0000-00005f690bf7"
