File: blocks/regulator_3v3.kicad_sch (KiCad schematic)
At the start: 3 parts, among them U501 TCR2EF 3.3V

Commit message: Updated references
Parts:
- renumbered C501 to C601, C505 to C605, U501 to U601
Changed lines of the file:
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@@
   (symbol (lib_id "Device:C_Small") (at 114.3 105.41 0) (unit 1)
     (in_bom yes) (on_board yes) (dnp no)
-    (property "Reference" "C501" (at 116.6368 104.2416 0)
+    (property "Reference" "C601" (at 116.6368 104.2416 0)
       (effects (font (size 1.27 1.27)) (justify left))
     )
@@
   (symbol (lib_id "Device:C_Small") (at 144.78 109.22 0) (unit 1)
     (in_bom yes) (on_board yes) (dnp no)
-    (property "Reference" "C505" (at 147.1168 108.0516 0)
+    (property "Reference" "C605" (at 147.1168 108.0516 0)
       (effects (font (size 1.27 1.27)) (justify left))
     )
@@
   (symbol (lib_id "KwanSystems:ADP122") (at 129.54 96.52 0) (unit 1)
     (in_bom yes) (on_board yes) (dnp no)
-    (property "Reference" "U501" (at 123.19 91.44 0)
+    (property "Reference" "U601" (at 123.19 91.44 0)
       (effects (font (size 1.27 1.27)) (justify left))
     )

Commit message: Update last 1.8V reference to 3.3V
Parts:
- C601: Purpose 1.8V Regulator Input -> 3.3V Regulator Input
- C605: Purpose 1.8V Regulator output -> 3.3V Regulator output
Changed lines of the file:
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@@
       (effects (font (size 1.27 1.27)) hide)
     )
-    (property "Purpose" "1.8V Regulator Input" (at 114.3 105.41 0)
+    (property "Purpose" "3.3V Regulator Input" (at 114.3 105.41 0)
       (effects (font (size 1.27 1.27)) hide)
     )
@@
     (instances
       (project "Precision23"
-        (path "/9151f981-b383-4946-8df4-92ef46ef2206/b677ca37-64a4-4c57-a7aa-64d766dbf7fc"
+        (path "/9151f981-b383-4946-8df4-92ef46ef2206/b9b5a9b9-9a45-4bb4-8a5d-f3809553447a/b677ca37-64a4-4c57-a7aa-64d766dbf7fc"
           (reference "C601") (unit 1)
         )
@@
       (effects (font (size 1.27 1.27)) hide)
     )
-    (property "Purpose" "1.8V Regulator output" (at 144.78 109.22 0)
+    (property "Purpose" "3.3V Regulator output" (at 144.78 109.22 0)
       (effects (font (size 1.27 1.27)) hide)
     )
@@
     (instances
       (project "Precision23"
-        (path "/9151f981-b383-4946-8df4-92ef46ef2206/b677ca37-64a4-4c57-a7aa-64d766dbf7fc"
+        (path "/9151f981-b383-4946-8df4-92ef46ef2206/b9b5a9b9-9a45-4bb4-8a5d-f3809553447a/b677ca37-64a4-4c57-a7aa-64d766dbf7fc"
           (reference "C605") (unit 1)
         )
@@
     (instances
       (project "Precision23"
-        (path "/9151f981-b383-4946-8df4-92ef46ef2206/b677ca37-64a4-4c57-a7aa-64d766dbf7fc"
+        (path "/9151f981-b383-4946-8df4-92ef46ef2206/b9b5a9b9-9a45-4bb4-8a5d-f3809553447a/b677ca37-64a4-4c57-a7aa-64d766dbf7fc"
           (reference "U601") (unit 1)
         )
