File: controllers/ATMEGA32U4.kicad_sch (KiCad schematic)
At the start: 12 parts, among them J1 USB_C2, U401 ATmega32U4-A, Y401 16MHz

Commit message: Added LED footprint with pins labeled A and C, to match legacy Precision
Parts:
- J1: footprint KwanSystems:USB4110 -> KwanSystems:GCTUSBTypeC_PTH
- R401: value 5.1k -> 22; footprint KwanSystems:R_Array_Convex_4x0402 -> Resistor_SMD:R_0603_1608Metric; symbol KwanSystems:RP4 -> KwanSystems:RESISTOR
- R401: footprint KwanSystems:R_Array_Convex_4x0402 -> Resistor_SMD:R_0603_1608Metric; symbol KwanSystems:RP4 -> KwanSystems:RESISTOR
- R408: value 330 -> 680; footprint KwanSystems:R_Array_Convex_2x0402 -> KwanSystems:R_Array_Convex_4x0402; symbol KwanSystems:RP2 -> KwanSystems:RP4
- U401: value ATmega32U4-A -> ATmega32U4; footprint Package_QFP:TQFP-44_10x10mm_P0.8mm -> Package_DFN_QFN:QFN-44-1EP_7x7mm_P0.5mm_EP5.2x5.2mm
Connections:
- net CC1: now also R401.1; no longer R401.4
- net CC2: no longer R401.3 (4)
- net CONN_D+: no longer R401.1 (4)
- net CONN_D-: no longer R401.2 (4)
- net D+: no longer R401.8 (5)
- net D-: no longer R401.7 (5)
- net GND: now also R401.2; no longer R401.5, R401.6 (5)
- net at D401.1 (K): now also R408.8 (5); no longer R408.4 (3)
- net ~{RESET}: now reaches S413.2, U401.13 (~{RESET})
- net at D402.1 (K): now also R408.7 (5); no longer R408.3
Other:
- moved on the sheet: R401
