File: controllers/ATMEGA32U4.kicad_sch (KiCad schematic)
At the start: 13 parts, among them U401 ATmega32U4-A, Y401 16MHz

Commit message: Updated references
Parts:
- removed R401: 22, Resistor_SMD:R_0603_1608Metric, symbol KwanSystems:RESISTOR
- R413: footprint Resistor_SMD:R_0402_1005Metric -> Resistor_SMD:R_0603_1608Metric
Connections:
- net D+: now also R403.2 (4); no longer R403.1 (4)
- net D-: now also R403.1 (4); no longer R403.2 (4)
- net Q_D+: now also R403.3; no longer R403.4 (3)
- net Q_D-: now also R403.4 (3); no longer R403.3
Other:
- moved on the sheet: R403A, R403B
Changed lines of the file:
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@@
       (effects (font (size 1.143 1.143)) (justify right))
     )
-    (property "Footprint" "Resistor_SMD:R_0402_1005Metric" (at 50.8 50.673 0)
+    (property "Footprint" "Resistor_SMD:R_0603_1608Metric" (at 50.8 50.673 0)
       (effects (font (size 0.508 0.508)) hide)
     )
@@
     )
   )
-  (symbol (lib_id "KwanSystems:RESISTOR") (at 50.8 90.17 0) (unit 2)
-    (in_bom yes) (on_board yes) (dnp no)
-    (property "Reference" "R401" (at 46.99 91.44 0)
-      (effects (font (size 1.143 1.143)))
-    )
-    (property "Value" "22" (at 54.61 91.44 0)
-      (effects (font (size 1.143 1.143)))
-    )
-    (property "Footprint" "Resistor_SMD:R_0603_1608Metric" (at 52.197 86.36 0)
-      (effects (font (size 0.508 0.508)) hide)
-    )
-    (property "Datasheet" "" (at 61.595 97.79 0)
-      (effects (font (size 1.524 1.524)) hide)
-    )
-    (pin "1")
-    (pin "2")
-    (instances
-      (project "Precision23"
-        (path "/9151f981-b383-4946-8df4-92ef46ef2206/bdd70cc5-4573-4ffd-a837-e689d69d580d"
-          (reference "R401") (unit 2)
-        )
-      )
-      (project "Naninator"
-        (path "/d855b238-2442-4e65-b657-8cbe334057c3/00000000-0000-0000-0000-00005964e4a0"
-          (reference "R403") (unit 1)
-        )
-      )
-    )
-  )
   (symbol (lib_id "Device:C_Small") (at 67.31 59.69 270) (unit 1)
     (in_bom yes) (on_board yes) (dnp no)
@@
     )
   )
-  (symbol (lib_id "KwanSystems:RP2") (at 67.31 85.09 0) (unit 2)
+  (symbol (lib_id "KwanSystems:RP2") (at 67.31 82.55 0) (unit 2)
+    (in_bom yes) (on_board yes) (dnp no)
+    (property "Reference" "R403" (at 62.23 81.28 0)
+      (effects (font (size 1.143 1.143)))
+    )
+    (property "Value" "22" (at 71.12 81.28 0)
+      (effects (font (size 1.143 1.143)))
+    )
+    (property "Footprint" "KwanSystems:R_Array_Convex_2x0402" (at 68.707 78.74 0)
+      (effects (font (size 0.508 0.508)) hide)
+    )
+    (property "Datasheet" "" (at 78.105 90.17 0)
+      (effects (font (size 1.524 1.524)) hide)
+    )
+    (pin "1")
+    (pin "4")
+    (pin "2")
+    (pin "3")
+    (instances
+      (project "Precision23"
+        (path "/9151f981-b383-4946-8df4-92ef46ef2206/bdd70cc5-4573-4ffd-a837-e689d69d580d"
+          (reference "R403") (unit 2)
+        )
+      )
+    )
+  )
+  (symbol (lib_id "Device:LED_Small") (at 165.1 149.86 90) (unit 1)
+    (in_bom yes) (on_board yes) (dnp no) (fields_autoplaced)
+    (property "Reference" "D402" (at 167.64 148.5265 90)
+      (effects (font (size 1.27 1.27)) (justify right))
+    )
+    (property "Value" "B" (at 167.64 151.0665 90)
+      (effects (font (size 1.27 1.27)) (justify right))
+    )
+    (property "Footprint" "LED_SMD:LED_0603_1608Metric" (at 165.1 149.86 90)
+      (effects (font (size 1.27 1.27)) hide)
+    )
+    (property "Datasheet" "~" (at 165.1 149.86 90)
+      (effects (font (size 1.27 1.27)) hide)
+    )
+    (property "Digikey" "754-1434-1-ND" (at 165.1 149.86 0)
+      (effects (font (size 1.27 1.27)) hide)
+    )
+    (property "Part Number" "APT1608QBC/D" (at 165.1 149.86 0)
+      (effects (font (size 1.27 1.27)) hide)
+    )
+    (pin "1")
+    (pin "2")
+    (instances
+      (project "Precision23"
+        (path "/9151f981-b383-4946-8df4-92ef46ef2206/bdd70cc5-4573-4ffd-a837-e689d69d580d"
+          (reference "D402") (unit 1)
+        )
+      )
+      (project "Naninator"
+        (path "/d855b238-2442-4e65-b657-8cbe334057c3/00000000-0000-0000-0000-00005964e4a0"
+          (reference "D402") (unit 1)
+        )
+      )
+    )
+  )
+  (symbol (lib_id "Device:C_Small") (at 67.31 67.31 90) (unit 1)
+    (in_bom yes) (on_board yes) (dnp no)
+    (property "Reference" "C416" (at 63.5 68.58 90)
+      (effects (font (size 1.27 1.27)))
+    )
+    (property "Value" "22pF" (at 71.12 68.58 90)
+      (effects (font (size 1.27 1.27)))
+    )
+    (property "Footprint" "Capacitor_SMD:C_0603_1608Metric" (at 67.31 67.31 0)
+      (effects (font (size 1.27 1.27)) hide)
+    )
+    (property "Datasheet" "~" (at 67.31 67.31 0)
+      (effects (font (size 1.27 1.27)) hide)
+    )
+    (pin "1")
+    (pin "2")
+    (instances
+      (project "Precision23"
+        (path "/9151f981-b383-4946-8df4-92ef46ef2206/bdd70cc5-4573-4ffd-a837-e689d69d580d"
+          (reference "C416") (unit 1)
+        )
+      )
+    )
+  )
+  (symbol (lib_id "KwanSystems:RP2") (at 67.31 85.09 0) (unit 1)
     (in_bom yes) (on_board yes) (dnp no)
     (property "Reference" "R403" (at 62.23 83.82 0)
@@
       (effects (font (size 1.524 1.524)) hide)
     )
-    (pin "1")
-    (pin "4")
-    (pin "2")
-    (pin "3")
-    (instances
-      (project "Precision23"
-        (path "/9151f981-b383-4946-8df4-92ef46ef2206/bdd70cc5-4573-4ffd-a837-e689d69d580d"
-          (reference "R403") (unit 2)
-        )
-      )
-    )
-  )
-  (symbol (lib_id "Device:LED_Small") (at 165.1 149.86 90) (unit 1)
-    (in_bom yes) (on_board yes) (dnp no) (fields_autoplaced)
-    (property "Reference" "D402" (at 167.64 148.5265 90)
-      (effects (font (size 1.27 1.27)) (justify right))
-    )
-    (property "Value" "B" (at 167.64 151.0665 90)
-      (effects (font (size 1.27 1.27)) (justify right))
-    )
-    (property "Footprint" "LED_SMD:LED_0603_1608Metric" (at 165.1 149.86 90)
-      (effects (font (size 1.27 1.27)) hide)
-    )
-    (property "Datasheet" "~" (at 165.1 149.86 90)
-      (effects (font (size 1.27 1.27)) hide)
-    )
-    (property "Digikey" "754-1434-1-ND" (at 165.1 149.86 0)
-      (effects (font (size 1.27 1.27)) hide)
-    )
-    (property "Part Number" "APT1608QBC/D" (at 165.1 149.86 0)
-      (effects (font (size 1.27 1.27)) hide)
-    )
-    (pin "1")
-    (pin "2")
-    (instances
-      (project "Precision23"
-        (path "/9151f981-b383-4946-8df4-92ef46ef2206/bdd70cc5-4573-4ffd-a837-e689d69d580d"
-          (reference "D402") (unit 1)
-        )
-      )
-      (project "Naninator"
-        (path "/d855b238-2442-4e65-b657-8cbe334057c3/00000000-0000-0000-0000-00005964e4a0"
-          (reference "D402") (unit 1)
-        )
-      )
-    )
-  )
-  (symbol (lib_id "Device:C_Small") (at 67.31 67.31 90) (unit 1)
-    (in_bom yes) (on_board yes) (dnp no)
-    (property "Reference" "C416" (at 63.5 68.58 90)
-      (effects (font (size 1.27 1.27)))
-    )
-    (property "Value" "22pF" (at 71.12 68.58 90)
-      (effects (font (size 1.27 1.27)))
-    )
-    (property "Footprint" "Capacitor_SMD:C_0603_1608Metric" (at 67.31 67.31 0)
-      (effects (font (size 1.27 1.27)) hide)
-    )
-    (property "Datasheet" "~" (at 67.31 67.31 0)
-      (effects (font (size 1.27 1.27)) hide)
-    )
-    (pin "1")
-    (pin "2")
-    (instances
-      (project "Precision23"
-        (path "/9151f981-b383-4946-8df4-92ef46ef2206/bdd70cc5-4573-4ffd-a837-e689d69d580d"
-          (reference "C416") (unit 1)
-        )
-      )
-    )
-  )
-  (symbol (lib_id "KwanSystems:RP2") (at 67.31 82.55 0) (unit 1)
-    (in_bom yes) (on_board yes) (dnp no)
-    (property "Reference" "R403" (at 62.23 81.28 0)
-      (effects (font (size 1.143 1.143)))
-    )
-    (property "Value" "22" (at 71.12 81.28 0)
-      (effects (font (size 1.143 1.143)))
-    )
-    (property "Footprint" "KwanSystems:R_Array_Convex_2x0402" (at 68.707 78.74 0)
-      (effects (font (size 0.508 0.508)) hide)
-    )
-    (property "Datasheet" "" (at 78.105 90.17 0)
-      (effects (font (size 1.524 1.524)) hide)
-    )
